File: PCB/PCB.sch (EAGLE design)
At the start: 17 parts, among them IC1 FT230XS, IC3 REG1117, X1 MINI-USB-32005-201

Commit message: v1.0 almost done
Parts:
- removed C4, C5: 22pF, microbuilder:CAP_CERAMIC0805-NOOUTLINE
- removed IC3: REG1117, burr-brown:REG1117
- removed QF1: 16M20AUM1, crystal:16M20AUM1
Connections:
- removed net XIN: C4.2, QF1.1
- removed net XOUT: C5.1, QF1.3
- new net SW1: IC2.9, S1.2
- new net SW2: IC2.10, S2.2
- net 3.3V: now also S1.1, S2.1, SV2.9; no longer IC3.VOUT
- net GND: no longer C4.1, C5.2, IC3.GND
- net RX: no longer IC2.3
- net TX: no longer IC2.4
- net UC_RX: now also IC2.3
- net UC_TX: now also IC2.4
- net VBAT: no longer IC3.VIN
Changed lines of the file:
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@@
 <part name="JP1" library="jumper" deviceset="JP2E" device=""/>
 <part name="JP2" library="jumper" deviceset="JP2E" device=""/>
-<part name="QF1" library="crystal" deviceset="16M20AUM1" device=""/>
-<part name="C4" library="microbuilder" deviceset="CAP_CERAMIC" device="0805-NOOUTLINE" value="22pF"/>
-<part name="C5" library="microbuilder" deviceset="CAP_CERAMIC" device="0805-NOOUTLINE" value="22pF"/>
-<part name="U$11" library="microbuilder" deviceset="GND" device=""/>
-<part name="U$12" library="microbuilder" deviceset="GND" device=""/>
 <part name="J1" library="SparkFun-Connectors" deviceset="JST_2MM_MALE" device=""/>
 <part name="U$10" library="microbuilder" deviceset="GND" device=""/>
-<part name="IC3" library="burr-brown" deviceset="REG1117" device=""/>
-<part name="U$8" library="microbuilder" deviceset="GND" device=""/>
 <part name="SV1" library="con-lstb" deviceset="MA03-1" device=""/>
 <part name="U$2" library="microbuilder" deviceset="GND" device=""/>
@@
 <instance part="JP1" gate="1" x="93.98" y="170.18"/>
 <instance part="JP2" gate="1" x="121.92" y="170.18"/>
-<instance part="QF1" gate="G$1" x="10.16" y="55.88" rot="R270"/>
-<instance part="C4" gate="G$1" x="10.16" y="63.5"/>
-<instance part="C5" gate="G$1" x="10.16" y="45.72"/>
-<instance part="U$11" gate="G$1" x="10.16" y="73.66" rot="R180"/>
-<instance part="U$12" gate="G$1" x="10.16" y="38.1"/>
 <instance part="J1" gate="G$1" x="12.7" y="170.18" rot="R90"/>
 <instance part="U$10" gate="G$1" x="27.94" y="162.56"/>
-<instance part="IC3" gate="G$1" x="27.94" y="137.16"/>
-<instance part="U$8" gate="G$1" x="27.94" y="119.38"/>
 <instance part="SV1" gate="G$1" x="15.24" y="106.68" rot="R270"/>
 <instance part="U$2" gate="G$1" x="17.78" y="91.44"/>
@@
 </segment>
 <segment>
-<pinref part="C4" gate="G$1" pin="1"/>
-<pinref part="U$11" gate="G$1" pin="GND"/>
-<wire x1="10.16" y1="71.12" x2="10.16" y2="68.58" width="0.1524" layer="91"/>
-</segment>
-<segment>
-<pinref part="C5" gate="G$1" pin="2"/>
-<pinref part="U$12" gate="G$1" pin="GND"/>
-<wire x1="10.16" y1="40.64" x2="10.16" y2="43.18" width="0.1524" layer="91"/>
-</segment>
-<segment>
 <pinref part="J1" gate="G$1" pin="-"/>
 <wire x1="17.78" y1="170.18" x2="27.94" y2="170.18" width="0.1524" layer="91"/>
@@
 </segment>
 <segment>
-<pinref part="IC3" gate="G$1" pin="GND"/>
-<pinref part="U$8" gate="G$1" pin="GND"/>
-<wire x1="27.94" y1="121.92" x2="27.94" y2="124.46" width="0.1524" layer="91"/>
-</segment>
-<segment>
 <pinref part="SV1" gate="G$1" pin="3"/>
 <pinref part="U$2" gate="G$1" pin="GND"/>
@@
 <net name="3.3V" class="0">
 <segment>
-<pinref part="IC3" gate="G$1" pin="VOUT"/>
-<wire x1="40.64" y1="137.16" x2="43.18" y2="137.16" width="0.1524" layer="91"/>
-<wire x1="43.18" y1="137.16" x2="43.18" y2="144.78" width="0.1524" layer="91"/>
-<label x="43.18" y="147.32" size="1.778" layer="95"/>
-</segment>
-<segment>
 <wire x1="93.98" y1="40.64" x2="93.98" y2="48.26" width="0.1524" layer="91"/>
 <label x="93.98" y="50.8" size="1.778" layer="95"/>
@@
 <pinref part="IC2" gate="G$1" pin="1"/>
 </segment>
+<segment>
+<pinref part="SV2" gate="1" pin="9"/>
+<wire x1="154.94" y1="172.72" x2="162.56" y2="172.72" width="0.1524" layer="91"/>
+<wire x1="162.56" y1="172.72" x2="162.56" y2="175.26" width="0.1524" layer="91"/>
+<label x="165.1" y="175.26" size="1.778" layer="95"/>
+</segment>
+<segment>
+<pinref part="S1" gate="G$1" pin="1"/>
+<wire x1="124.46" y1="71.12" x2="137.16" y2="71.12" width="0.1524" layer="91"/>
+<wire x1="137.16" y1="71.12" x2="137.16" y2="76.2" width="0.1524" layer="91"/>
+<label x="137.16" y="78.74" size="1.778" layer="95"/>
+</segment>
+<segment>
+<pinref part="S2" gate="G$1" pin="1"/>
+<wire x1="124.46" y1="63.5" x2="137.16" y2="63.5" width="0.1524" layer="91"/>
+<wire x1="137.16" y1="63.5" x2="137.16" y2="66.04" width="0.1524" layer="91"/>
+<label x="137.16" y="66.04" size="1.778" layer="95"/>
+</segment>
 </net>
 <net name="TX" class="0">
+<segment>
+<pinref part="SV2" gate="1" pin="5"/>
+<wire x1="154.94" y1="162.56" x2="162.56" y2="162.56" width="0.1524" layer="91"/>
+<label x="162.56" y="165.1" size="1.778" layer="95"/>
+</segment>
 <segment>
 <pinref part="JP1" gate="1" pin="2"/>
@@
 <label x="91.44" y="157.48" size="1.778" layer="95"/>
 </segment>
-<segment>
-<pinref part="SV2" gate="1" pin="5"/>
-<wire x1="154.94" y1="162.56" x2="162.56" y2="162.56" width="0.1524" layer="91"/>
-<label x="162.56" y="165.1" size="1.778" layer="95"/>
-</segment>
-<segment>
-<wire x1="53.34" y1="33.02" x2="40.64" y2="33.02" width="0.1524" layer="91"/>
-<label x="38.1" y="30.48" size="1.778" layer="95"/>
-<pinref part="IC2" gate="G$1" pin="4"/>
-</segment>
 </net>
 <net name="RX" class="0">
+<segment>
+<pinref part="SV2" gate="1" pin="4"/>
+<wire x1="154.94" y1="160.02" x2="162.56" y2="160.02" width="0.1524" layer="91"/>
+<label x="162.56" y="160.02" size="1.778" layer="95"/>
+</segment>
 <segment>
 <pinref part="JP2" gate="1" pin="2"/>
 <wire x1="121.92" y1="167.64" x2="121.92" y2="160.02" width="0.1524" layer="91"/>
 <label x="121.92" y="157.48" size="1.778" layer="95"/>
-</segment>
-<segment>
-<pinref part="SV2" gate="1" pin="4"/>
-<wire x1="154.94" y1="160.02" x2="162.56" y2="160.02" width="0.1524" layer="91"/>
-<label x="162.56" y="160.02" size="1.778" layer="95"/>
-</segment>
-<segment>
-<wire x1="53.34" y1="35.56" x2="40.64" y2="35.56" width="0.1524" layer="91"/>
-<label x="38.1" y="35.56" size="1.778" layer="95"/>
-<pinref part="IC2" gate="G$1" pin="3"/>
 </segment>
 </net>
@@
 <net name="UC_RX" class="0">
 <segment>
+<wire x1="53.34" y1="35.56" x2="40.64" y2="35.56" width="0.1524" layer="91"/>
+<label x="38.1" y="35.56" size="1.778" layer="95"/>
+<pinref part="IC2" gate="G$1" pin="3"/>
+</segment>
+<segment>
 <pinref part="JP1" gate="1" pin="3"/>
 <wire x1="96.52" y1="167.64" x2="96.52" y2="165.1" width="0.1524" layer="91"/>
@@
 <net name="UC_TX" class="0">
 <segment>
+<wire x1="53.34" y1="33.02" x2="40.64" y2="33.02" width="0.1524" layer="91"/>
+<label x="38.1" y="30.48" size="1.778" layer="95"/>
+<pinref part="IC2" gate="G$1" pin="4"/>
+</segment>
+<segment>
 <pinref part="JP2" gate="1" pin="3"/>
 <wire x1="124.46" y1="167.64" x2="124.46" y2="162.56" width="0.1524" layer="91"/>
 <label x="127" y="160.02" size="1.778" layer="95"/>
-</segment>
-</net>
-<net name="XIN" class="0">
-<segment>
-<wire x1="20.32" y1="58.42" x2="17.78" y2="58.42" width="0.1524" layer="91"/>
-<wire x1="17.78" y1="58.42" x2="15.24" y2="60.96" width="0.1524" layer="91"/>
-<wire x1="15.24" y1="60.96" x2="10.16" y2="60.96" width="0.1524" layer="91"/>
-<pinref part="QF1" gate="G$1" pin="1"/>
-<wire x1="10.16" y1="60.96" x2="10.16" y2="58.42" width="0.1524" layer="91"/>
-<pinref part="C4" gate="G$1" pin="2"/>
-<junction x="10.16" y="60.96"/>
-<label x="20.32" y="60.96" size="1.778" layer="95"/>
-</segment>
-</net>
-<net name="XOUT" class="0">
-<segment>
-<wire x1="17.78" y1="53.34" x2="15.24" y2="50.8" width="0.1524" layer="91"/>
-<wire x1="15.24" y1="50.8" x2="10.16" y2="50.8" width="0.1524" layer="91"/>
-<pinref part="QF1" gate="G$1" pin="3"/>
-<wire x1="10.16" y1="50.8" x2="10.16" y2="53.34" width="0.1524" layer="91"/>
-<pinref part="C5" gate="G$1" pin="1"/>
-<junction x="10.16" y="50.8"/>
-<wire x1="17.78" y1="53.34" x2="20.32" y2="53.34" width="0.1524" layer="91"/>
-<label x="20.32" y="48.26" size="1.778" layer="95"/>
 </segment>
 </net>
@@
 </segment>
 <segment>
-<pinref part="IC3" gate="G$1" pin="VIN"/>
-<wire x1="15.24" y1="137.16" x2="10.16" y2="137.16" width="0.1524" layer="91"/>
-<wire x1="10.16" y1="137.16" x2="10.16" y2="144.78" width="0.1524" layer="91"/>
-<label x="10.16" y="147.32" size="1.778" layer="95"/>
-</segment>
-<segment>
 <pinref part="SV2" gate="1" pin="2"/>
 <wire x1="154.94" y1="154.94" x2="167.64" y2="154.94" width="0.1524" layer="91"/>
 <wire x1="167.64" y1="154.94" x2="167.64" y2="170.18" width="0.1524" layer="91"/>
-<label x="170.18" y="172.72" size="1.778" layer="95"/>
+<label x="170.18" y="170.18" size="1.778" layer="95"/>
 </segment>
 </net>
@@
 </segment>
 </net>
+<net name="SW1" class="0">
+<segment>
+<pinref part="S1" gate="G$1" pin="2"/>
+<wire x1="114.3" y1="71.12" x2="101.6" y2="71.12" width="0.1524" layer="91"/>
+<wire x1="101.6" y1="71.12" x2="101.6" y2="78.74" width="0.1524" layer="91"/>
+<label x="99.06" y="81.28" size="1.778" layer="95"/>
+</segment>
+<segment>
+<pinref part="IC2" gate="G$1" pin="9"/>
+<wire x1="53.34" y1="20.32" x2="45.72" y2="20.32" width="0.1524" layer="91"/>
+<label x="43.18" y="20.32" size="1.778" layer="95"/>
+</segment>
+</net>
+<net name="SW2" class="0">
+<segment>
+<pinref part="S2" gate="G$1" pin="2"/>
+<wire x1="114.3" y1="63.5" x2="101.6" y2="63.5" width="0.1524" layer="91"/>
+<wire x1="101.6" y1="63.5" x2="101.6" y2="68.58" width="0.1524" layer="91"/>
+<label x="96.52" y="68.58" size="1.778" layer="95"/>
+</segment>
+<segment>
+<pinref part="IC2" gate="G$1" pin="10"/>
+<wire x1="53.34" y1="17.78" x2="45.72" y2="17.78" width="0.1524" layer="91"/>
+<label x="43.18" y="17.78" size="1.778" layer="95"/>
+</segment>
+</net>
